Commit message: Re-organized repo for better clarity

File: my_robot_description/urdf/mobile_base_gazebo.xacro (robot description, xacro)
@@ -2,10 +2,10 @@
 <robot name="my_robot" xmlns:xacro="http://www.ros.org/wiki/xacro">
     <gazebo reference="right_wheel_link">
-        <mu1 value="0.3" />
-        <mu2 value="0.3" />
+        <mu1 value="1.0" />
+        <mu2 value="1.0" />
     </gazebo>
     <gazebo reference="left_wheel_link">
-        <mu1 value="0.3" />
-        <mu2 value="0.3" />
+        <mu1 value="1.0" />
+        <mu2 value="1.0" />
     </gazebo>
     <gazebo reference="caster_wheel_link">

File: my_robot_description/urdf/my_robot.urdf.xacro (robot description, xacro)
@@ -6,9 +6,9 @@
     <xacro:include filename="mobile_base_gazebo.xacro" />
     <xacro:include filename="camera.xacro" />
-    <xacro:include filename="standalone_arm.urdf.xacro" />
+    <!-- <xacro:include filename="standalone_arm.urdf.xacro" />
     <joint name="mobile_base_arm_base_joint" type="fixed">
         <parent link="base_link" />
         <child link="arm_base_link" />
         <origin xyz="${base_length / 4.0} 0 ${base_height}" rpy="0 0 0"/>
-    </joint>
+    </joint> -->
 </robot>
