Commit message: Completed MoveIt Course + organized repo more

File: course_level2/my_robot_description/urdf/my_robot.urdf.xacro (robot description, xacro)
@@ -6,9 +6,9 @@
     <xacro:include filename="mobile_base_gazebo.xacro" />
     <xacro:include filename="camera.xacro" />
-    <!-- <xacro:include filename="standalone_arm.urdf.xacro" />
+    <xacro:include filename="standalone_arm.urdf.xacro" />
     <joint name="mobile_base_arm_base_joint" type="fixed">
         <parent link="base_link" />
         <child link="arm_base_link" />
         <origin xyz="${base_length / 4.0} 0 ${base_height}" rpy="0 0 0"/>
-    </joint> -->
+    </joint>
 </robot>

Commit message: Adding ros2_control, README not updated.

File: course_level2/my_robot_description/urdf/my_robot.urdf.xacro (robot description, xacro)
@@ -6,9 +6,9 @@
     <xacro:include filename="mobile_base_gazebo.xacro" />
     <xacro:include filename="camera.xacro" />
-    <xacro:include filename="standalone_arm.urdf.xacro" />
-    <joint name="mobile_base_arm_base_joint" type="fixed">
+    <!-- <xacro:include filename="standalone_arm.urdf.xacro" /> -->
+    <!-- <joint name="mobile_base_arm_base_joint" type="fixed">
         <parent link="base_link" />
         <child link="arm_base_link" />
         <origin xyz="${base_length / 4.0} 0 ${base_height}" rpy="0 0 0"/>
-    </joint>
+    </joint> -->
 </robot>
