Commit message: ros2_control add

File: course_ros2_control/base_robot_description/urdf/base_robot.urdf.xacro (robot description, xacro)
@@ -3,4 +3,11 @@
     <xacro:include filename="common_properties.xacro" />
     <xacro:include filename="mobile_base.xacro" />
-    <xacro:include filename="mobile_base.ros2_control.xacro" />
+    <!-- <xacro:include filename="mobile_base.ros2_control.xacro" /> -->
+    <xacro:include filename="arm.ros2_control.xacro" />
+    <xacro:include filename="arm.xacro" />
+    <joint name="mobile_base_arm_base_joint" type="fixed">
+        <parent link="base_link" />
+        <child link="arm_base_link" />
+        <origin xyz="${base_length / 4.0} 0 ${base_height}" rpy="0 0 0"/>
+    </joint>
 </robot>

File: course_ros2_control/base_robot_description/urdf/common_properties.xacro (robot description, xacro)
@@ -2,8 +2,41 @@
 <robot xmlns:xacro="http://www.ros.org/wiki/xacro">
     <material name="blue">
-        <color rgba="0 0 0.5 1" />
+        <color rgba="0.10 0.35 1.0 1" /> <!-- r g b alpha -->
     </material>
     <material name="grey">
-        <color rgba="0.5 0.5 0.5 1" />
+        <color rgba="0.5 0.5 0.5 1" /> <!-- r g b alpha -->
     </material>
+    <material name="orange">
+        <color rgba="1.00 0.38 0.02 1" /> <!-- r g b alpha -->
+    </material>
+    <material name="yellow">
+        <color rgba="1.0 0.65 0.1  1" /> <!-- r g b alpha -->
+    </material>
+    <xacro:macro name="box_inertia" params="m x y z o_xyz o_rpy">
+        <inertial>
+            <mass value="${m}" />
+            <origin xyz="${o_xyz}" rpy="${o_rpy}" />
+            <inertia ixx="${(m/12) * (y*y + z*z)}" ixy="0" ixz="0"
+                     iyy="${(m/12) * (x*x + z*z)}" iyz="0"
+                     izz="${(m/12) * (y*y + x*x)}" />
+        </inertial>
+    </xacro:macro>
+    <xacro:macro name="cylinder_inertia" params="m r h o_xyz o_rpy">
+        <inertial>
+            <mass value="${m}" />
+            <origin xyz="${o_xyz}" rpy="${o_rpy}" />
+            <inertia ixx="${(m/12) * (3*r*r + h*h)}" ixy="0" ixz="0"
+                     iyy="${(m/12) * (3*r*r + h*h)}" iyz="0"
+                     izz="${(m/2) * (r*r)}" />
+        </inertial>
+    </xacro:macro>
+    <xacro:macro name="sphere_inertia" params="m r o_xyz o_rpy">
+        <inertial>
+            <mass value="${m}" />
+            <origin xyz="${o_xyz}" rpy="${o_rpy}" />
+            <inertia ixx="${(2/5) * m * r*r}" ixy="0" ixz="0"
+                     iyy="${(2/5) * m * r*r}" iyz="0"
+                     izz="${(2/5) * m * r*r}" />
+        </inertial>
+    </xacro:macro>
 </robot>

File: course_ros2_control/base_robot_description/urdf/mobile_base.ros2_control.xacro (robot description, xacro)
@@ -5,5 +5,9 @@
             <plugin>mock_components/GenericSystem</plugin>
             <param name="calculate_dynamics">true</param>
+            <!-- We can only run the line below instead of controller above if we have hardware -->
             <!-- <plugin>mobile_base_hardware/MobileBaseHardwareInterface</plugin> -->
+            <param name="left_motor_id">10</param>
+            <param name="right_motor_id">20</param>
+            <param name="dynamixel_port">/dev/ttyACM0</param>
         </hardware>
         <joint name="base_right_wheel_joint">
